File: kicad/817-TTL-Serial-Optoisolator.kicad_pcb (KiCad board)
At the start: 2 copper layers, 40.6 x 22.9 mm, 17 parts, among them P1 CONN_4, P2 CONN_4, Q1 2N3906, Q2 2N3906, U1 817, U2 817

Commit message: initial release
Other:
- board text added: "817 TTL Serial Optoisolator v1"
- board text removed: "TTL Serial Optoisolator v1"
Changed lines of the file:
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@@
     (links 20)
     (no_connects 0)
-    (area 199.339999 52.019999 240.080001 74.980001)
+    (area 198.5264 50.673 240.8936 76.073)
     (thickness 1.6)
     (drawings 27)
@@
   )
   (setup
-    (last_trace_width 0.508)
+    (last_trace_width 0.254)
     (user_trace_width 0.508)
     (trace_clearance 0.254)
@@
     (effects (font (size 0.635 0.635) (thickness 0.127)) (justify mirror))
   )
-  (gr_text "TTL Serial Optoisolator v1" (at 219.71 53.34) (layer B.SilkS)
+  (gr_text "817 TTL Serial Optoisolator v1" (at 219.71 53.34) (layer B.SilkS)
     (effects (font (size 1.016 1.016) (thickness 0.2032)) (justify mirror))
   )
@@
     (effects (font (size 0.762 0.762) (thickness 0.1524)) (justify right))
   )
-  (segment (start 228.6 60.96) (end 228.6 60.325) (width 0.508) (layer F.Cu) (net 3) (status C00000))
-  (segment (start 229.87 59.055) (end 229.87 57.15) (width 0.508) (layer F.Cu) (net 3) (status 800000))
-  (segment (start 228.6 60.325) (end 229.87 59.055) (width 0.508) (layer F.Cu) (net 3) (status 400000))
-  (segment (start 231.14 60.96) (end 231.14 60.325) (width 0.508) (layer F.Cu) (net 4) (status C00000))
-  (segment (start 229.87 54.61) (end 228.6 55.88) (width 0.508) (layer F.Cu) (net 4) (status 800000))
+  (segment (start 228.6 60.96) (end 228.6 60.325) (width 0.508) (layer F.Cu) (net 3))
+  (segment (start 229.87 59.055) (end 229.87 57.15) (width 0.508) (layer F.Cu) (net 3))
+  (segment (start 228.6 60.325) (end 229.87 59.055) (width 0.508) (layer F.Cu) (net 3))
+  (segment (start 231.14 60.96) (end 231.14 60.325) (width 0.508) (layer F.Cu) (net 4))
+  (segment (start 229.87 54.61) (end 228.6 55.88) (width 0.508) (layer F.Cu) (net 4))
   (segment (start 231.14 54.61) (end 229.87 54.61) (width 0.508) (layer F.Cu) (net 4))
   (segment (start 232.41 55.88) (end 231.14 54.61) (width 0.508) (layer F.Cu) (net 4))
   (segment (start 232.41 56.515) (end 232.41 55.88) (width 0.508) (layer F.Cu) (net 4))
   (segment (start 232.41 59.055) (end 232.41 56.515) (width 0.508) (layer F.Cu) (net 4))
-  (segment (start 231.14 60.325) (end 232.41 59.055) (width 0.508) (layer F.Cu) (net 4) (status 400000))
+  (segment (start 231.14 60.325) (end 232.41 59.055) (width 0.508) (layer F.Cu) (net 4))
   (segment (start 223.52 60.96) (end 228.6 66.04) (width 0.508) (layer F.Cu) (net 5))
   (segment (start 228.6 66.04) (end 228.6 71.12) (width 0.508) (layer F.Cu) (net 5))
   (segment (start 210.82 55.88) (end 210.82 60.96) (width 0.508) (layer F.Cu) (net 6))
   (segment (start 210.82 60.96) (end 215.9 66.04) (width 0.508) (layer F.Cu) (net 6))
-  (segment (start 208.28 66.04) (end 207.01 67.31) (width 0.508) (layer F.Cu) (net 7) (status 400000))
-  (segment (start 209.55 72.39) (end 210.82 71.12) (width 0.508) (layer F.Cu) (net 7) (status 800000))
+  (segment (start 208.28 66.04) (end 207.01 67.31) (width 0.508) (layer F.Cu) (net 7))
+  (segment (start 209.55 72.39) (end 210.82 71.12) (width 0.508) (layer F.Cu) (net 7))
   (segment (start 208.28 72.39) (end 209.55 72.39) (width 0.508) (layer F.Cu) (net 7))
   (segment (start 207.01 71.12) (end 208.28 72.39) (width 0.508) (layer F.Cu) (net 7))
@@
   (segment (start 213.36 55.88) (end 212.09 54.61) (width 0.508) (layer F.Cu) (net 9))
   (segment (start 209.55 56.515) (end 209.55 55.245) (width 0.254) (layer F.Cu) (net 9))
-  (segment (start 203.2 64.77) (end 201.93 64.77) (width 0.508) (layer F.Cu) (net 9) (status 800000))
+  (segment (start 203.2 64.77) (end 201.93 64.77) (width 0.508) (layer F.Cu) (net 9))
   (segment (start 209.55 54.61) (end 209.55 55.245) (width 0.508) (layer F.Cu) (net 9))
   (segment (start 210.185 53.975) (end 209.55 54.61) (width 0.508) (layer F.Cu) (net 9))
@@
   (segment (start 214.63 60.96) (end 215.9 60.96) (width 0.508) (layer F.Cu) (net 9))
   (segment (start 201.93 64.77) (end 201.93 64.135) (width 0.254) (layer F.Cu) (net 9))
-  (segment (start 226.06 71.12) (end 226.06 72.39) (width 0.508) (layer F.Cu) (net 10) (status 400000))
-  (segment (start 233.68 68.58) (end 237.49 64.77) (width 0.508) (layer F.Cu) (net 10) (status 800000))
+  (segment (start 226.06 71.12) (end 226.06 72.39) (width 0.508) (layer F.Cu) (net 10))
+  (segment (start 233.68 68.58) (end 237.49 64.77) (width 0.508) (layer F.Cu) (net 10))
   (segment (start 233.68 71.755) (end 233.68 68.58) (width 0.508) (layer F.Cu) (net 10))
   (segment (start 232.41 73.025) (end 233.68 71.755) (width 0.508) (layer F.Cu) (net 10))
   (segment (start 226.695 73.025) (end 232.41 73.025) (width 0.508) (layer F.Cu) (net 10))
   (segment (start 226.06 72.39) (end 226.695 73.025) (width 0.508) (layer F.Cu) (net 10))
-  (segment (start 226.06 71.12) (end 226.06 67.31) (width 0.508) (layer F.Cu) (net 10) (status 400000))
-  (segment (start 224.79 66.04) (end 223.52 66.04) (width 0.508) (layer F.Cu) (net 10) (status 800000))
+  (segment (start 226.06 71.12) (end 226.06 67.31) (width 0.508) (layer F.Cu) (net 10))
+  (segment (start 224.79 66.04) (end 223.52 66.04) (width 0.508) (layer F.Cu) (net 10))
   (segment (start 226.06 67.31) (end 224.79 66.04) (width 0.508) (layer F.Cu) (net 10))
   (segment (start 208.28 55.88) (end 201.93 62.23) (width 0.508) (layer F.Cu) (net 11))
@@
   (segment (start 206.375 64.135) (end 205.74 64.77) (width 0.508) (layer F.Cu) (net 13))
   (segment (start 201.93 59.69) (end 200.66 60.96) (width 0.508) (layer F.Cu) (net 13))
-  (segment (start 212.09 64.77) (end 213.36 66.04) (width 0.508) (layer F.Cu) (net 13) (status 800000))
+  (segment (start 212.09 64.77) (end 213.36 66.04) (width 0.508) (layer F.Cu) (net 13))
   (segment (start 204.47 66.04) (end 205.74 64.77) (width 0.508) (layer F.Cu) (net 13))
   (segment (start 203.2 66.04) (end 204.47 66.04) (width 0.508) (layer F.Cu) (net 13))
@@
   (segment (start 226.06 60.96) (end 227.33 62.23) (width 0.508) (layer F.Cu) (net 14))
   (segment (start 227.33 62.23) (end 227.965 62.865) (width 0.508) (layer F.Cu) (net 14))
-  (segment (start 234.95 59.69) (end 237.49 59.69) (width 0.508) (layer F.Cu) (net 14) (status 800000))
+  (segment (start 234.95 59.69) (end 237.49 59.69) (width 0.508) (layer F.Cu) (net 14))
   (segment (start 231.775 62.865) (end 234.95 59.69) (width 0.508) (layer F.Cu) (net 14))
-  (segment (start 226.06 60.96) (end 226.06 60.325) (width 0.508) (layer F.Cu) (net 14) (status C00000))
-  (segment (start 227.33 59.055) (end 227.33 57.15) (width 0.508) (layer F.Cu) (net 14) (status 800000))
-  (segment (start 226.06 60.325) (end 227.33 59.055) (width 0.508) (layer F.Cu) (net 14) (status 400000))
+  (segment (start 226.06 60.96) (end 226.06 60.325) (width 0.508) (layer F.Cu) (net 14))
+  (segment (start 227.33 59.055) (end 227.33 57.15) (width 0.508) (layer F.Cu) (net 14))
+  (segment (start 226.06 60.325) (end 227.33 59.055) (width 0.508) (layer F.Cu) (net 14))
   (zone (net 1) (net_name GNDA) (layer B.Cu) (hatch edge 0.508)
     (connect_pads (clearance 0.508))
